File: kicad/Maytal.kicad_pcb (KiCad board)
At the start: 2 copper layers, 94.1 x 94.7 mm, 11 parts, among them IC1 ArduinoProMini, P1 LIPO_SOLAR, P2 CONN_01X03, Q1 PN2222A, U1 FONA_808, U2 Adafruit_DS3231

Commit message: Rerouted power bus
Parts:
- moved P1 2.60 mm to (123.3, 80.0), turned to 0 degrees
Connections:
- P1 pad 1: RAW -> Net-(P1-Pad1)
- P1 pad 2: GND -> Net-(P1-Pad2)
Routing:
- net RAW: track 63.8 -> 32.5 mm
Other:
- board text added: "Pressure Telemetry v0.3"
- board text removed: "Pressure Telemetry v0.1"
